File: pcbs/CAN bus transceiver v2 PYBv11/CAN bus transceiver v2 PYBv11.kicad_pcb (KiCad board)
At the start: 2 copper layers, 30.6 x 40.6 mm, 20 parts, among them P1 CONN_01X16, P2 CONN_01X02, P3 CONN_01X16, P4 CONN_01X02, Q1 Q_PMOS_SGD, U1 TCAN337GDR, U2 TCAN337GDR, U3 LM3489

Commit message: can: changed Zenner diode footprint
Parts:
- D1: footprint Diodes_SMD:SMB_Handsoldering -> Diodes_SMD:SOD-523
- moved D1 2.70 mm to (87.0, 106.7)
Changed lines of the file:
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@@
     (links 49)
     (no_connects 23)
-    (area 81.839999 90.094999 112.470001 121.360001)
+    (area 81.839999 90.094999 112.597001 130.885001)
     (thickness 1.6)
     (drawings 17)
@@
     )
   )
-  (module Diodes_SMD:SMB_Handsoldering (layer F.Cu)
-    (at 89.662 107.188)
-    (descr "Diode SMB Handsoldering")
-    (tags "Diode SMB Handsoldering")
-    (attr smd)
-    (fp_text reference D1 (at 0 -3.1) (layer F.SilkS)
-      (effects (font (size 1 1) (thickness 0.15)))
-    )
-    (fp_text value ZENER (at 0.1 4.75) (layer F.Fab)
-      (effects (font (size 1 1) (thickness 0.15)))
-    )
-    (fp_line (start -4.7 -2.25) (end 4.7 -2.25) (layer F.CrtYd) (width 0.05))
-    (fp_line (start 4.7 -2.25) (end 4.7 2.25) (layer F.CrtYd) (width 0.05))
-    (fp_line (start 4.7 2.25) (end -4.7 2.25) (layer F.CrtYd) (width 0.05))
-    (fp_line (start -4.7 2.25) (end -4.7 -2.25) (layer F.CrtYd) (width 0.05))
-    (fp_line (start -0.44958 0) (end 0.39878 -1.00076) (layer F.SilkS) (width 0.15))
-    (fp_line (start 0.39878 -1.00076) (end 0.39878 1.00076) (layer F.SilkS) (width 0.15))
-    (fp_line (start 0.39878 1.00076) (end -0.44958 0) (layer F.SilkS) (width 0.15))
-    (fp_line (start -0.44958 0) (end -0.44958 1.00076) (layer F.SilkS) (width 0.15))
-    (fp_line (start -0.44958 0) (end -0.44958 -1.00076) (layer F.SilkS) (width 0.15))
-    (fp_text user K (at -3.5 3.1) (layer F.SilkS)
-      (effects (font (size 1 1) (thickness 0.15)))
-    )
-    (fp_text user A (at 3 3.05) (layer F.SilkS)
-      (effects (font (size 1 1) (thickness 0.15)))
-    )
-    (fp_line (start -2.30632 1.8) (end -2.30632 1.6002) (layer F.SilkS) (width 0.15))
-    (fp_line (start -1.84928 1.8) (end -1.84928 1.601) (layer F.SilkS) (width 0.15))
-    (fp_line (start 2.30124 1.8) (end 2.30124 1.651) (layer F.SilkS) (width 0.15))
-    (fp_line (start -2.30124 -1.8) (end -2.30124 -1.651) (layer F.SilkS) (width 0.15))
-    (fp_line (start -1.84928 -1.8) (end -1.84928 -1.651) (layer F.SilkS) (width 0.15))
-    (fp_line (start 2.30124 -1.8) (end 2.30124 -1.651) (layer F.SilkS) (width 0.15))
-    (fp_line (start -1.84928 1.94898) (end -1.84928 1.75086) (layer F.SilkS) (width 0.15))
-    (fp_line (start -1.84928 -1.99898) (end -1.84928 -1.80086) (layer F.SilkS) (width 0.15))
-    (fp_line (start 2.29616 1.99644) (end 2.29616 1.79832) (layer F.SilkS) (width 0.15))
-    (fp_line (start -2.30632 1.99644) (end 2.29616 1.99644) (layer F.SilkS) (width 0.15))
-    (fp_line (start -2.30632 1.99644) (end -2.30632 1.79832) (layer F.SilkS) (width 0.15))
-    (fp_line (start -2.30124 -1.99898) (end -2.30124 -1.80086) (layer F.SilkS) (width 0.15))
-    (fp_line (start -2.30124 -1.99898) (end 2.30124 -1.99898) (layer F.SilkS) (width 0.15))
-    (fp_line (start 2.30124 -1.99898) (end 2.30124 -1.80086) (layer F.SilkS) (width 0.15))
-    (pad 1 smd rect (at -2.70002 0) (size 3.50012 2.30124) (layers F.Cu F.Paste F.Mask)
-      (net 9 +12V))
-    (pad 2 smd rect (at 2.70002 0) (size 3.50012 2.30124) (layers F.Cu F.Paste F.Mask)
-      (net 7 GND))
-    (model Diodes_SMD.3dshapes/SMB_Handsoldering.wrl
-      (at (xyz 0 0 0))
-      (scale (xyz 0.3937 0.3937 0.3937))
-      (rotate (xyz 0 0 180))
-    )
-  )
   (module Inductors:Inductor_Taiyo-Yuden_NR-80xx_HandSoldering (layer F.Cu)
     (at 90.7415 125.9205 180)
@@
     )
   )
+  (module Diodes_SMD:SOD-523 (layer F.Cu)
+    (at 86.995 106.7435)
+    (descr "http://www.diodes.com/datasheets/ap02001.pdf p.144")
+    (tags "Diode SOD523")
+    (attr smd)
+    (fp_text reference D1 (at 0 -1.5) (layer F.SilkS)
+      (effects (font (size 1 1) (thickness 0.15)))
+    )
+    (fp_text value ZENER (at 0 1.7) (layer F.Fab)
+      (effects (font (size 1 1) (thickness 0.15)))
+    )
+    (fp_line (start 1.25 -0.75) (end 1.25 0.75) (layer F.CrtYd) (width 0.05))
+    (fp_line (start -1.25 -0.75) (end 1.25 -0.75) (layer F.CrtYd) (width 0.05))
+    (fp_line (start -1.25 0.75) (end -1.25 -0.75) (layer F.CrtYd) (width 0.05))
+    (fp_line (start 1.25 0.75) (end -1.25 0.75) (layer F.CrtYd) (width 0.05))
+    (fp_line (start 0.1 0) (end 0.25 0) (layer F.Fab) (width 0.15))
+    (fp_line (start 0.1 -0.2) (end -0.2 0) (layer F.Fab) (width 0.15))
+    (fp_line (start 0.1 0.2) (end 0.1 -0.2) (layer F.Fab) (width 0.15))
+    (fp_line (start -0.2 0) (end 0.1 0.2) (layer F.Fab) (width 0.15))
+    (fp_line (start -0.2 0) (end -0.35 0) (layer F.Fab) (width 0.15))
+    (fp_line (start -0.2 0.2) (end -0.2 -0.2) (layer F.Fab) (width 0.15))
+    (fp_line (start 0.6 -0.4) (end 0.6 0.4) (layer F.Fab) (width 0.15))
+    (fp_line (start -0.6 -0.4) (end 0.6 -0.4) (layer F.Fab) (width 0.15))
+    (fp_line (start -0.6 0.4) (end -0.6 -0.4) (layer F.Fab) (width 0.15))
+    (fp_line (start 0.6 0.4) (end -0.6 0.4) (layer F.Fab) (width 0.15))
+    (fp_line (start 0.6 -0.6) (end -1 -0.6) (layer F.SilkS) (width 0.15))
+    (fp_line (start 0.6 0.6) (end -1 0.6) (layer F.SilkS) (width 0.15))
+    (pad 2 smd rect (at 0.7 0 180) (size 0.6 0.7) (layers F.Cu F.Paste F.Mask)
+      (net 7 GND))
+    (pad 1 smd rect (at -0.7 0 180) (size 0.6 0.7) (layers F.Cu F.Paste F.Mask)
+      (net 9 +12V))
+  )
   (gr_line (start 112.522 90.17) (end 81.915 90.17) (angle 90) (layer Edge.Cuts) (width 0.15))
